File: Skematik Main Compressor V1/Skematik Main Compressor V1/HUMADITY.kicad_sch (KiCad schematic)
At the start: 3 parts, among them J6 Conn_01x06_Socket

Commit message: Penambahan Skematik Main Compressor V1
Parts:
- J6: value Conn_01x06_Socket -> SHT31
Connections:
- net VCC is gone; now on net 3.3V: J6.1 (Pin_1)
- net INT: no longer names the net of J6.5 (Pin_5)
- no-connect marks 1 -> 2
Changed lines of the file:
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@@
+	)
+	(no_connect
+		(at 148.59 104.14)
 	)
 	(no_connect
@@
 	(wire
 		(pts
-			(xy 137.16 104.14) (xy 148.59 104.14)
-		)
-		(stroke
-			(width 0)
-			(type default)
-		)
-	)
-	(wire
-		(pts
 			(xy 139.7 99.06) (xy 148.59 99.06)
 		)
@@
 		)
 	)
-	(hierarchical_label "VCC"
+	(hierarchical_label "3.3V"
 		(shape input)
 		(at 137.16 93.98 180)
-		(fields_autoplaced yes)
-		(effects
-			(font
-				(size 1.27 1.27)
-			)
-			(justify right)
-		)
-	)
-	(hierarchical_label "INT"
-		(shape input)
-		(at 137.16 104.14 180)
 		(fields_autoplaced yes)
 		(effects
@@
 			)
 		)
-		(property "Value" "Conn_01x06_Socket"
+		(property "Value" "SHT31"
 			(at 154.94 101.5999 0)
 			(effects
