File: Skematik Main Compressor V1/Skematik Main Compressor V1/RELAY.kicad_sch (KiCad schematic)
At the start: 7 parts, among them J5 Conn_01x03_Pin, K2 SANYOU_SRD_Form_C, Q2 2N5551-TA, U4 PC817

Commit message: Penambahan Skematik Main Compressor V1
Parts:
- removed J5: Conn_01x03_Pin, Connector_PinHeader_2.54mm:PinHeader_1x03_P2.54mm_Vertical, symbol Connector:Conn_01x03_Pin
- removed Q2: 2N5551-TA, symbol 2N5551-TA:2N5551-TA
- removed R11, R12: R, Resistor_SMD:R_0603_1608Metric_Pad0.98x0.95mm_HandSolder, symbol Device:R
- added Q7: 2N5551-TA, Custom-Library-FRES:TO-92-Wide-Inline, symbol Custom Simbol FRES:2N5551-TA
- added R11: 1K, Resistor_SMD:R_0402_1005Metric_Pad0.72x0.64mm_HandSolder, symbol Device:R_US
- added R12: 510, Resistor_SMD:R_0402_1005Metric_Pad0.72x0.64mm_HandSolder, symbol Device:R_US
Connections:
- net GND: now also Q7.3 (E)
- net PIN D: now also R11.1
- net at U4.1: now also R11.2
- net at K2.2: now also Q7.1 (C)
- net at U4.3: now also R12.1
- net VOLT renamed VDD
- new net: Q7.2 (B), R12.2
