File: Skematik Main Compressor V1/Skematik Main Compressor V1/RELAY.kicad_sch (KiCad schematic)
At the start: 6 parts, among them K4 SANYOU_SRD_Form_C, Q7 2N5551-TA, U11 PC817

Commit message: menghapus file tidak perlu
Parts:
- removed Q7: 2N5551-TA, Custom-Library-FRES:TO-92-Wide-Inline, symbol Custom Simbol FRES:2N5551-TA
- added Q3: 2N5551-TA, Package_TO_SOT_THT:TO-92_Inline_Wide, symbol Custom Simbol FRES:2N5551-TA
Connections:
- net GND: now also Q3.3 (E)
- net at K4.2: now also Q3.1 (C)
- net at R29.2: now also Q3.2 (B)
Changed lines of the file:
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@@
 		(dnp no)
 		(fields_autoplaced yes)
-		(property "Reference" "Q7"
+		(property "Reference" "Q3"
 			(at 132.08 104.1399 0)
 			(effects
@@
 			)
 		)
-		(property "Footprint" "Custom-Library-FRES:TO-92-Wide-Inline"
+		(property "Footprint" "Package_TO_SOT_THT:TO-92_Inline_Wide"
 			(at 190.5 105.41 0)
 			(effects
@@
 			)
 		)
+		(pin "2"
+		)
 		(pin "3"
-		)
-		(pin "2"
 		)
 		(pin "1"
 		)
 		(instances
-			(project ""
+			(project "Skematik Main Compressor V1"
 				(path "/04b6c12f-837a-46bf-a4f1-2bcc73eb17c7/461449bc-6630-4ddb-8246-b2b959924c81"
-					(reference "Q7")
+					(reference "Q4")
 					(unit 1)
 				)
 				(path "/04b6c12f-837a-46bf-a4f1-2bcc73eb17c7/4c793412-26aa-466b-acda-2c0eafce3a9b"
-					(reference "Q6")
+					(reference "Q3")
 					(unit 1)
 				)
