File: Skematik Main Compressor V1/Skematik Main Compressor V1/Relay Motor1.kicad_sch (KiCad schematic)
At the start: 7 parts, among them J2 Conn_01x03_Pin, K1 SANYOU_SRD_Form_C, Q1 2N5551-TA, U2 PC817

Commit message: Penambahan Skematik Main Compressor V1
Parts:
- removed J2: Conn_01x03_Pin, Connector_PinHeader_2.54mm:PinHeader_1x03_P2.54mm_Vertical, symbol Connector:Conn_01x03_Pin
- removed R1, R2: R, Resistor_SMD:R_0603_1608Metric_Pad0.98x0.95mm_HandSolder, symbol Device:R
- added R1: 1K, Resistor_SMD:R_0402_1005Metric_Pad0.72x0.64mm_HandSolder, symbol Device:R_US
- added R15: 510, Resistor_SMD:R_0402_1005Metric_Pad0.72x0.64mm_HandSolder, symbol Device:R_US
Connections:
- net PIN D: now also R1.1
- net at Q1.2 (B): now also R15.2
- net at U2.1: now also R1.2
- net at U2.3: now also R15.1
