File: Skematik Main Compressor V1/Skematik Main Compressor V1/Skematik Main Compressor V1.kicad_sch (KiCad schematic)
At the start: 16 parts, among them J1 UART, J12 Boot, J13 IN 12V, J15 MOTOR1, J16 MOTOR2, J17 AUTO DRAIN, J18 Buzzer AC, J19 JUMPER, J2 MOTOR IN, U1 ESP32-WROOM-32UE

Commit message: Update baru skematik main
Other:
- note added: "AC TRIP"
- note added: "AUTO DRAIN"
- note added: "BUZER DC"
- note added: "F-ram"
- note added: "LCD"
- note added: "LORA"
- note added: "RELAY BUZER AC"
- note added: "RELAY MOTOR 1"
- note added: "RELAY MOTOR 2"
- note added: "RTC"
- note added: "Regulator DC"
- note added: "SDCARD"
- note added: "SENSOR HUMADITY"
- note added: "SENSOR PREASURE & CO"
Changed lines of the file:
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@@
+		)
+	)
+	(text "RELAY MOTOR 1"
+		(exclude_from_sim no)
+		(at 214.63 64.77 0)
+		(effects
+			(font
+				(size 1.27 1.27)
+			)
 		)
 	)
@@
 		(exclude_from_sim no)
 		(at 167.64 54.61 0)
+		(effects
+			(font
+				(size 1.27 1.27)
+			)
+		)
+	)
+	(text "LORA"
+		(exclude_from_sim no)
+		(at 260.985 109.855 0)
+		(effects
+			(font
+				(size 1.27 1.27)
+			)
+		)
+	)
+	(text "BUZER DC"
+		(exclude_from_sim no)
+		(at 78.105 65.405 0)
 		(effects
 			(font
@@
 		)
 	)
+	(text "SENSOR PREASURE & CO "
+		(exclude_from_sim no)
+		(at 167.005 18.415 0)
+		(effects
+			(font
+				(size 1.27 1.27)
+			)
+		)
+	)
+	(text "F-ram\n"
+		(exclude_from_sim no)
+		(at 77.47 20.32 0)
+		(effects
+			(font
+				(size 1.27 1.27)
+			)
+		)
+	)
 	(text "Address 0x45 (Solder)\n\n"
 		(exclude_from_sim no)
 		(at 259.715 52.705 0)
+		(effects
+			(font
+				(size 1.27 1.27)
+			)
+		)
+	)
+	(text "RTC"
+		(exclude_from_sim no)
+		(at 215.265 20.955 0)
+		(effects
+			(font
+				(size 1.27 1.27)
+			)
+		)
+	)
+	(text "LCD"
+		(exclude_from_sim no)
+		(at 124.46 20.955 0)
+		(effects
+			(font
+				(size 1.27 1.27)
+			)
+		)
+	)
+	(text "AUTO DRAIN"
+		(exclude_from_sim no)
+		(at 169.545 65.405 0)
+		(effects
+			(font
+				(size 1.27 1.27)
+			)
+		)
+	)
+	(text "RELAY BUZER AC"
+		(exclude_from_sim no)
+		(at 123.19 65.405 0)
+		(effects
+			(font
+				(size 1.27 1.27)
+			)
+		)
+	)
+	(text "AC TRIP"
+		(exclude_from_sim no)
+		(at 31.115 65.405 0)
+		(effects
+			(font
+				(size 1.27 1.27)
+			)
+		)
+	)
+	(text "SDCARD"
+		(exclude_from_sim no)
+		(at 214.63 109.855 0)
+		(effects
+			(font
+				(size 1.27 1.27)
+			)
+		)
+	)
+	(text "Regulator DC"
+		(exclude_from_sim no)
+		(at 33.02 19.685 0)
+		(effects
+			(font
+				(size 1.27 1.27)
+			)
+		)
+	)
+	(text "SENSOR HUMADITY\n"
+		(exclude_from_sim no)
+		(at 259.08 20.32 0)
 		(effects
 			(font
@@
 		(effects
 			(font
+				(size 1.27 1.27)
+			)
+		)
+	)
+	(text "RELAY MOTOR 2"
+		(exclude_from_sim no)
+		(at 258.445 64.135 0)
+		(effects
+			(font
