File: Skematik Main Compressor V1/Skematik Main Compressor V1/stc.kicad_sch (KiCad schematic)
At the start: 5 parts, among them U2 DS3231M

Commit message: Penambahan Skematik Main Compressor V1
Parts:
- removed C1: 100nF, Capacitor_SMD:C_0402_1005Metric_Pad0.74x0.62mm_HandSolder, symbol Device:C
- removed R3, R4: 4K7, Resistor_THT:R_Axial_DIN0204_L3.6mm_D1.6mm_P5.08mm_Horizontal, symbol Device:R
- removed U2: DS3231M, Package_SO:SOIC-16W_7.5x10.3mm_P1.27mm, symbol Timer_RTC:DS3231M
- added C12: 100nF, Capacitor_SMD:C_0402_1005Metric_Pad0.74x0.62mm_HandSolder, symbol Device:C
- added R7, R8: 4K7, Resistor_SMD:R_0402_1005Metric_Pad0.72x0.64mm_HandSolder, symbol Device:R_US
- added U7: DS3231M, Package_SO:SOIC-16W_7.5x10.3mm_P1.27mm, symbol Timer_RTC:DS3231M
Connections:
- net 3.3V: now also R7.1, R8.1, U7.2 (VCC)
- net GND: now also C12.2, U7.10 (GND), U7.11 (GND), U7.12 (GND), U7.13 (GND), U7.5 (GND), U7.6 (GND), U7.7 (GND), U7.8 (GND), U7.9 (GND)
- net SCL: now also R8.2, U7.16 (SCL)
- net SDA: now also R7.2, U7.15 (SDA)
- net at BAT1.1 (+): now also C12.1, U7.14 (VBAT)
Other:
- note removed: "Addres RTCds3231 : 0x68"
