File: Skematik Main Compressor V1/Skematik Main Compressor V1/stc.kicad_sch (KiCad schematic)
At the start: 5 parts, among them U7 DS3231M

Commit message: menghapus file tidak perlu
Parts:
- removed BAT1: ~, Custom-Library-FRES:1056TR, symbol Custom Simbol FRES:Battery_Cell_CR1220
- added BT1: CR1220MFR_FH, CR1220:CR1220-SMD, symbol CR1220MFR_FH:CR1220MFR_FH
Connections:
- net GND: now also BT1.2 (-)
- net at C12.1, U7.14 (VBAT): now also BT1.1 (+)
Other:
- moved on the sheet: C12
Changed lines of the file:
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@@
+	(wire
+		(pts
+			(xy 175.26 85.09) (xy 175.26 87.63)
+		)
+		(stroke
+			(width 0)
+			(type default)
+		)
+	)
 	(wire
 		(pts
@@
 	(wire
 		(pts
+			(xy 163.83 86.995) (xy 163.83 85.09)
+		)
+		(stroke
+			(width 0)
+			(type default)
+		)
+	)
+	(wire
+		(pts
 			(xy 129.54 97.79) (xy 129.54 100.33)
 		)
@@
 	(wire
 		(pts
-			(xy 163.83 92.71) (xy 163.83 96.52)
+			(xy 163.83 94.615) (xy 163.83 96.52)
 		)
 		(stroke
@@
 	(wire
 		(pts
-			(xy 175.26 92.71) (xy 175.26 96.52)
+			(xy 175.26 90.17) (xy 175.26 96.52)
 		)
 		(stroke
@@
 	(symbol
 		(lib_id "Device:C")
-		(at 163.83 88.9 0)
+		(at 163.83 90.805 0)
 		(unit 1)
 		(exclude_from_sim no)
@@
 		(dnp no)
 		(property "Reference" "C12"
-			(at 166.37 87.63 0)
+			(at 166.37 89.535 0)
 			(effects
 				(font
@@
 		)
 		(property "Value" "100nF"
-			(at 166.37 90.17 0)
+			(at 166.37 92.075 0)
 			(effects
 				(font
@@
 		)
 		(property "Footprint" "Capacitor_SMD:C_0402_1005Metric_Pad0.74x0.62mm_HandSolder"
-			(at 164.7952 92.71 0)
+			(at 164.7952 94.615 0)
 			(effects
 				(font
@@
 		)
 		(property "Datasheet" "~"
-			(at 163.83 88.9 0)
+			(at 163.83 90.805 0)
 			(effects
 				(font
@@
 		)
 		(property "Description" "Unpolarized capacitor"
-			(at 163.83 88.9 0)
+			(at 163.83 90.805 0)
 			(effects
 				(font
@@
 	)
 	(symbol
-		(lib_id "Custom Simbol FRES:Battery_Cell_CR1220")
-		(at 175.26 88.9 0)
+		(lib_id "CR1220MFR_FH:CR1220MFR_FH")
+		(at 175.26 90.17 0)
+		(mirror x)
 		(unit 1)
 		(exclude_from_sim no)
@@
 		(on_board yes)
 		(dnp no)
-		(fields_autoplaced yes)
-		(property "Reference" "BAT1"
-			(at 179.07 87.6934 0)
-			(effects
-				(font
-					(size 1.27 1.27)
-				)
-				(justify left)
-			)
-		)
-		(property "Value" "~"
-			(at 179.07 89.5985 0)
-			(effects
-				(font
-					(size 1.27 1.27)
-				)
-				(justify left)
-			)
-		)
-		(property "Footprint" "Custom-Library-FRES:1056TR"
-			(at 175.26 88.9 0)
-			(effects
-				(font
-					(size 1.27 1.27)
-				)
-				(hide yes)
-			)
-		)
-		(property "Datasheet" ""
-			(at 175.26 88.9 0)
-			(effects
-				(font
-					(size 1.27 1.27)
-				)
-				(hide yes)
-			)
-		)
-		(property "Description" ""
-			(at 175.26 88.9 0)
-			(effects
-				(font
-					(size 1.27 1.27)
-				)
-				(hide yes)
-			)
+		(property "Reference" "BT1"
+			(at 191.77 90.1701 0)
+			(effects
+				(font
+					(size 1.27 1.27)
+				)
+				(justify left)
+			)
+		)
+		(property "Value" "CR1220MFR_FH"
+			(at 191.77 87.6301 0)
+			(effects
+				(font
+					(size 1.27 1.27)
+				)
+				(justify left)
+			)
+		)
+		(property "Footprint" "CR1220:CR1220-SMD"
+			(at 191.77 -4.75 0)
+			(effects
+				(font
+					(size 1.27 1.27)
+				)
+				(justify left top)
+				(hide yes)
+			)
+		)
+		(property "Datasheet" "https://www.renatabatteries.us/sites/default/files/2018-01/CR1220MFR-FH.pdf"
+			(at 191.77 -104.75 0)
+			(effects
+				(font
+					(size 1.27 1.27)
+				)
+				(justify left top)
+				(hide yes)
+			)
+		)
+		(property "Description" "Coin Cell Battery 3V2-PINHORZ40mAh"
+			(at 175.26 90.17 0)
+			(effects
+				(font
+					(size 1.27 1.27)
+				)
+				(hide yes)
+			)
+		)
+		(property "Height" "2.95"
+			(at 191.77 -304.75 0)
+			(effects
+				(font
+					(size 1.27 1.27)
+				)
+				(justify left top)
+				(hide yes)
+			)
+		)
+		(property "Mouser Part Number" "614-CR1220MFR-FH"
+			(at 191.77 -404.75 0)
+			(effects
+				(font
+					(size 1.27 1.27)
+				)
+				(justify left top)
+				(hide yes)
+			)
+		)
+		(property "Mouser Price/Stock" "https://www.mouser.co.uk/ProductDetail/Renata/CR1220MFR-FH?qs=PuikTf%252BlMsxvBg0JpoIdQQ%3D%3D"
+			(at 191.77 -504.75 0)
+			(effects
+				(font
+					(size 1.27 1.27)
+				)
+				(justify left top)
+				(hide yes)
+			)
+		)
+		(property "Manufacturer_Name" "RENATA"
+			(at 191.77 -604.75 0)
+			(effects
+				(font
+					(size 1.27 1.27)
+				)
+				(justify left top)
+				(hide yes)
+			)
+		)
+		(property "Manufacturer_Part_Number" "CR1220MFR FH"
+			(at 191.77 -704.75 0)
+			(effects
+				(font
+					(size 1.27 1.27)
+				)
+				(justify left top)
+				(hide yes)
+			)
+		)
+		(pin "2"
 		)
 		(pin "1"
-		)
-		(pin "2"
 		)
 		(instances
 			(project ""
 				(path "/04b6c12f-837a-46bf-a4f1-2bcc73eb17c7/71c25820-6749-41c5-9e93-e0d91d28a35c"
-					(reference "BAT1")
+					(reference "BT1")
 					(unit 1)
 				)
