File: Skematik Main Compressor V1/Skematik Main Compressor V1/LORA.kicad_sch (KiCad schematic)
At the start: 1 part, among them U3 RA-02_LORA

Commit message: Penambahan Skematik Main Compressor V1
Connections:
- net 3V3 renamed 3.3V
Changed lines of the file:
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@@
 		)
 	)
-	(hierarchical_label "3V3"
+	(hierarchical_label "3.3V"
 		(shape input)
 		(at 156.21 85.09 0)

Commit message: menghapus file tidak perlu
Parts:
- U3: footprint RA-02_LORA:MODULE_RA-02_LORA -> RF_Module:Ai-Thinker-Ra-01-LoRa
Changed lines of the file:
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@@
 			)
 		)
-		(property "Footprint" "RA-02_LORA:MODULE_RA-02_LORA"
+		(property "Footprint" "RF_Module:Ai-Thinker-Ra-01-LoRa"
 			(at 135.89 97.79 0)
 			(effects
