File: Skematik Main Compressor V1/Skematik Main Compressor V1/Regulator dc.kicad_sch (KiCad schematic)
At the start: 8 parts, among them U5 LM1117DT-3.3, U6 LM2576S-5

Commit message: menghapus file tidak perlu
Changed lines of the file:
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@@
-	)
-	(junction
-		(at 92.71 78.74)
-		(diameter 0)
-		(color 0 0 0 0)
 	)
 	(junction
@@
 	)
 	(junction
-		(at 173.99 85.09)
-		(diameter 0)
-		(color 0 0 0 0)
-	)
-	(junction
 		(at 185.42 74.93)
 		(diameter 0)
@@
 	)
 	(junction
-		(at 146.05 85.09)
-		(diameter 0)
-		(color 0 0 0 0)
-	)
-	(junction
 		(at 101.6 69.85)
 		(diameter 0)
@@
 	(wire
 		(pts
+			(xy 101.6 78.74) (xy 101.6 79.375)
+		)
+		(stroke
+			(width 0)
+			(type default)
+		)
+	)
+	(wire
+		(pts
 			(xy 101.6 69.85) (xy 101.6 73.66)
 		)
@@
 	(wire
 		(pts
+			(xy 82.55 78.74) (xy 82.55 79.375)
+		)
+		(stroke
+			(width 0)
+			(type default)
+		)
+	)
+	(wire
+		(pts
 			(xy 173.99 74.93) (xy 175.26 74.93)
 		)
@@
 	(wire
 		(pts
-			(xy 173.99 85.09) (xy 185.42 85.09)
-		)
-		(stroke
-			(width 0)
-			(type default)
-		)
-	)
-	(wire
-		(pts
 			(xy 78.74 69.85) (xy 82.55 69.85)
 		)
@@
 	(wire
 		(pts
+			(xy 100.33 69.85) (xy 101.6 69.85)
+		)
+		(stroke
+			(width 0)
+			(type default)
+		)
+	)
+	(wire
+		(pts
 			(xy 173.99 83.82) (xy 173.99 85.09)
 		)
@@
 	(wire
 		(pts
-			(xy 146.05 85.09) (xy 146.05 87.63)
-		)
-		(stroke
-			(width 0)
-			(type default)
-		)
-	)
-	(wire
-		(pts
-			(xy 146.05 85.09) (xy 173.99 85.09)
-		)
-		(stroke
-			(width 0)
-			(type default)
-		)
-	)
-	(wire
-		(pts
-			(xy 92.71 77.47) (xy 92.71 78.74)
-		)
-		(stroke
-			(width 0)
-			(type default)
-		)
-	)
-	(wire
-		(pts
-			(xy 100.33 69.85) (xy 101.6 69.85)
+			(xy 146.05 80.01) (xy 146.05 87.63)
 		)
 		(stroke
@@
 	(wire
 		(pts
-			(xy 146.05 80.01) (xy 146.05 85.09)
-		)
-		(stroke
-			(width 0)
-			(type default)
-		)
-	)
-	(wire
-		(pts
-			(xy 92.71 78.74) (xy 101.6 78.74)
-		)
-		(stroke
-			(width 0)
-			(type default)
-		)
-	)
-	(wire
-		(pts
-			(xy 92.71 78.74) (xy 92.71 81.28)
+			(xy 92.71 77.47) (xy 92.71 81.28)
 		)
 		(stroke
@@
 	(wire
 		(pts
-			(xy 82.55 78.74) (xy 92.71 78.74)
-		)
-		(stroke
-			(width 0)
-			(type default)
-		)
-	)
-	(wire
-		(pts
 			(xy 132.08 69.85) (xy 135.89 69.85)
 		)
@@
 		(pts
 			(xy 82.55 69.85) (xy 85.09 69.85)
-		)
-		(stroke
-			(width 0)
-			(type default)
-		)
-	)
-	(wire
-		(pts
-			(xy 135.89 85.09) (xy 146.05 85.09)
 		)
 		(stroke
@@
 		)
 	)
+	(hierarchical_label "GND"
+		(shape input)
+		(at 101.6 79.375 270)
+		(fields_autoplaced yes)
+		(effects
+			(font
+				(size 1.27 1.27)
+			)
+			(justify right)
+		)
+	)
 	(hierarchical_label "3.3V"
 		(shape input)
@@
 		)
 	)
+	(hierarchical_label "GND"
+		(shape input)
+		(at 135.89 85.09 270)
+		(fields_autoplaced yes)
+		(effects
+			(font
+				(size 1.27 1.27)
+			)
+			(justify right)
+		)
+	)
+	(hierarchical_label "GND"
+		(shape input)
+		(at 82.55 79.375 270)
+		(fields_autoplaced yes)
+		(effects
+			(font
+				(size 1.27 1.27)
+			)
+			(justify right)
+		)
+	)
+	(hierarchical_label "GND"
+		(shape input)
+		(at 185.42 85.09 270)
+		(fields_autoplaced yes)
+		(effects
+			(font
+				(size 1.27 1.27)
+			)
+			(justify right)
+		)
+	)
 	(hierarchical_label "12V"
 		(shape input)
@@
 	(hierarchical_label "GND"
 		(shape input)
-		(at 146.05 87.63 0)
-		(fields_autoplaced yes)
-		(effects
-			(font
-				(size 1.27 1.27)
-			)
-			(justify left)
-		)
-	)
+		(at 173.99 85.09 270)
+		(fields_autoplaced yes)
+		(effects
+			(font
+				(size 1.27 1.27)
+			)
+			(justify right)
+		)
+	)
+	(hierarchical_label "GND"
+		(shape input)
+		(at 146.05 87.63 270)
+		(fields_autoplaced yes)
+		(effects
+			(font
+				(size 1.27 1.27)
+			)
+			(justify right)
+		)
+	)
