File: Skematik Main Compressor V1/Skematik Main Compressor V1/SDcard.kicad_sch (KiCad schematic)
At the start: 7 parts, among them J3 MSD-4-A

Commit message: Penambahan Skematik Main Compressor V1
Parts:
- removed R3, R4, R5, R6: 10k, Resistor_SMD:R_0402_1005Metric_Pad0.72x0.64mm_HandSolder, symbol Device:R
- added R3, R4, R5, R6: 10K, Resistor_SMD:R_0402_1005Metric_Pad0.72x0.64mm_HandSolder, symbol Device:R_US
Connections:
- net +3.3V: now also R3.1, R4.2, R5.2, R6.2
- net CLK: now also R5.1
- net MISO: now also R6.1
- net MOSI: now also R4.1
- net CS renamed CD
- net CD: now also R3.2

Commit message: menghapus file tidak perlu
Parts:
- J3: footprint MSD4A -> MSD-4-A:CUI_MSD-4-A
