File: Skematik Main Compressor V1/Skematik Main Compressor V1/Skematik Main Compressor V1.kicad_pcb (KiCad board)
At the start: 2 copper layers, 40 parts, among them J1 Conn_01x04_Pin, J2 Conn_01x03_Pin, J5 Conn_01x03_Pin, J6 Conn_01x06_Socket, J7 ADS1015, J8 PREASURE SENSOR, J9 CO SENSOR, K1 SANYOU_SRD_Form_C, K2 SANYOU_SRD_Form_C, U1 ESP32-WROOM-32UE, U2 PC817, U3 RA-02_LORA, U4 PC817, U5 LM1117DT-3.3, U6 LM2576S-5, U7 DS3231M

Commit message: Update baru skematik main
Parts:
- removed J5: Conn_01x03_Pin, Connector_PinHeader_2.54mm:PinHeader_1x03_P2.54mm_Vertical
- added BZ1: Buzzer, Buzzer_Beeper:Buzzer_12x9.5RM7.6, F.Cu at (-62.7, 165.4)
- added C10: C_Polarized_US, Capacitor_SMD:CP_Elec_3x5.3, F.Cu at (-117.3, 179.3)
- added C12: 100nF, Capacitor_SMD:C_0402_1005Metric_Pad0.74x0.62mm_HandSolder, F.Cu at (-53.2, 136.2)
- added C9: C_Polarized_US, Capacitor_SMD:CP_Elec_3x5.3, F.Cu at (-117.3, 174.4)
- added D10: TRIP 1, LED_SMD:LED_0201_0603Metric_Pad0.64x0.40mm_HandSolder, F.Cu at (-116.9, 163.0)
- added D11: TRIP 2, LED_SMD:LED_0201_0603Metric_Pad0.64x0.40mm_HandSolder, F.Cu at (-116.9, 164.7)
- added D12: MERAH, LED_SMD:LED_0402_1005Metric_Pad0.77x0.64mm_HandSolder, F.Cu at (-97.8, 146.0)
- added D13: BIRU, LED_SMD:LED_0402_1005Metric_Pad0.77x0.64mm_HandSolder, F.Cu at (-97.8, 148.0)
- added D4: LED, LED_SMD:LED_0805_2012Metric_Pad1.15x1.40mm_HandSolder, F.Cu at (-75.5, 177.1)
- added D5: LED, LED_SMD:LED_0805_2012Metric_Pad1.15x1.40mm_HandSolder, F.Cu at (-98.7, 177.1)
- added D6: MB6S, Package_TO_SOT_SMD:TO-269AA, F.Cu at (-125.0, 175.2)
- added D7: MB6S, Package_TO_SOT_SMD:TO-269AA, F.Cu at (-125.0, 181.5)
- added D8: D_Schottky_Small_Filled, Diode_SMD:D_0201_0603Metric_Pad0.64x0.40mm_HandSolder, F.Cu at (-116.9, 159.5)
- added D9: D_Schottky_Small_Filled, Diode_SMD:D_0201_0603Metric_Pad0.64x0.40mm_HandSolder, F.Cu at (-116.9, 161.2)
- added J12: Boot, Connector_PinHeader_2.54mm:PinHeader_1x02_P2.54mm_Vertical, F.Cu at (-96.1, 137.7)
- added J13: IN 12V, Connector_Molex:Molex_KK-396_A-41791-0002_1x02_P3.96mm_Vertical, F.Cu at (144.5, 74.5)
- added J15: MOTOR1, Connector_Molex:Molex_KK-396_A-41791-0002_1x02_P3.96mm_Vertical, F.Cu at (19.1, 145.5)
- added J16: MOTOR2, Connector_Molex:Molex_KK-396_A-41791-0002_1x02_P3.96mm_Vertical, F.Cu at (19.1, 84.0)
- added J17: AUTO DRAIN, Connector_Molex:Molex_KK-396_A-41791-0002_1x02_P3.96mm_Vertical, F.Cu at (19.0, 104.5)
- added J18: Buzzer AC, Connector_Molex:Molex_KK-396_A-41791-0002_1x02_P3.96mm_Vertical, F.Cu at (19.0, 121.0)
- added J19: JUMPER, Connector_PinHeader_2.54mm:PinHeader_1x03_P2.54mm_Vertical, F.Cu at (52.5, 86.4)
- added J4: Conn_01x04_Pin, Connector_JST:JST_EH_B4B-EH-A_1x04_P2.50mm_Vertical, F.Cu at (-66.6, 207.4)
- added K3: SANYOU_SRD_Form_C, Relay_THT:Relay_SPDT_SANYOU_SRD_Series_Form_C, F.Cu at (28.5, 81.5)
- added K4: SANYOU_SRD_Form_C, Relay_THT:Relay_SPDT_SANYOU_SRD_Series_Form_C, F.Cu at (28.0, 102.5)
- added Q5: BC547, Package_TO_SOT_THT:TO-92_Inline_Wide, F.Cu at (-64.1, 175.4)
- added R10: 1k8, Resistor_THT:R_Axial_DIN0204_L3.6mm_D1.6mm_P5.08mm_Horizontal, F.Cu at (-56.5, 149.4)
- added R15: 510, Resistor_SMD:R_0402_1005Metric_Pad0.72x0.64mm_HandSolder, F.Cu at (-120.2, 206.6)
- added R16: 510, Resistor_SMD:R_0402_1005Metric_Pad0.72x0.64mm_HandSolder, F.Cu at (-71.5, 178.5)
- added R17: 1K, Resistor_SMD:R_0402_1005Metric_Pad0.72x0.64mm_HandSolder, F.Cu at (-94.7, 176.5)
- added R18: 1K, Resistor_SMD:R_0402_1005Metric_Pad0.72x0.64mm_HandSolder, F.Cu at (-101.5, 151.3)
- added R19: 1k, Resistor_SMD:R_0402_1005Metric_Pad0.72x0.64mm_HandSolder, F.Cu at (-55.9, 173.1)
- added R20: 150K, Resistor_THT:R_Axial_DIN0204_L3.6mm_D1.6mm_P5.08mm_Horizontal, F.Cu at (-135.9, 160.2)
- added R21: 150K, Resistor_THT:R_Axial_DIN0204_L3.6mm_D1.6mm_P5.08mm_Horizontal, F.Cu at (-135.9, 163.3)
- added R22: 10k, Resistor_THT:R_Axial_DIN0204_L3.6mm_D1.6mm_P5.08mm_Horizontal, F.Cu at (-135.9, 166.5)
- added R23: 10k, Resistor_THT:R_Axial_DIN0204_L3.6mm_D1.6mm_P5.08mm_Horizontal, F.Cu at (-135.9, 169.6)
- added R24: 10k, Resistor_THT:R_Axial_DIN0204_L3.6mm_D1.6mm_P5.08mm_Horizontal, F.Cu at (-135.9, 172.8)
- added R25: 10k, Resistor_THT:R_Axial_DIN0204_L3.6mm_D1.6mm_P5.08mm_Horizontal, F.Cu at (-135.9, 175.9)
- added R26: 10K, Resistor_SMD:R_0402_1005Metric_Pad0.72x0.64mm_HandSolder, F.Cu at (-82.6, 201.5)
- added R27: 10K, Resistor_SMD:R_0402_1005Metric_Pad0.72x0.64mm_HandSolder, F.Cu at (-82.6, 203.5)
- added R28: 1K, Resistor_SMD:R_0402_1005Metric_Pad0.72x0.64mm_HandSolder, F.Cu at (-101.5, 153.3)
- added R29: 510, Resistor_SMD:R_0402_1005Metric_Pad0.72x0.64mm_HandSolder, F.Cu at (-94.7, 178.5)
- added R9: 1k8, Resistor_SMD:R_0402_1005Metric_Pad0.72x0.64mm_HandSolder, F.Cu at (-48.4, 148.8)
- added U10: PC817, Package_DIP:DIP-4_W7.62mm, F.Cu at (-87.2, 177.6)
- added U11: PC817, Package_DIP:DIP-4_W7.62mm, F.Cu at (-110.3, 177.6)
- added U12: PC817, Package_DIP:DIP-4_W7.62mm, F.Cu at (-127.8, 160.7)
- added U13: PC817, Package_DIP:DIP-4_W7.62mm, F.Cu at (-127.8, 167.4)
- added U9: FM24C64B, Package_SO:SOIC-8_3.9x4.9mm_P1.27mm, F.Cu at (-53.8, 144.6)
- J1: value Conn_01x04_Pin -> UART
- J2: value Conn_01x03_Pin -> MOTOR IN; footprint Connector_PinHeader_2.54mm:PinHeader_1x03_P2.54mm_Vertical -> Connector_Molex:Molex_KK-396_A-41791-0003_1x03_P3.96mm_Vertical
- J6: value Conn_01x06_Socket -> SHT31
- R1, R11, R2: value R -> 1K; footprint Resistor_SMD:R_0603_1608Metric_Pad0.98x0.95mm_HandSolder -> Resistor_SMD:R_0402_1005Metric_Pad0.72x0.64mm_HandSolder
- R12: value R -> 510; footprint Resistor_SMD:R_0603_1608Metric_Pad0.98x0.95mm_HandSolder -> Resistor_SMD:R_0402_1005Metric_Pad0.72x0.64mm_HandSolder
- R3, R4, R5, R6: value 10k -> 10K
- R7, R8: footprint Resistor_THT:R_Axial_DIN0204_L3.6mm_D1.6mm_P5.08mm_Horizontal -> Resistor_SMD:R_0402_1005Metric_Pad0.72x0.64mm_HandSolder
- moved R1 301.2 mm to (-120.2, 204.6)
- moved D1 292.3 mm to (-124.2, 205.2)
- moved U2 292.3 mm to (-135.8, 205.7)
- moved R2 243.7 mm to (-71.5, 176.5)
- moved R11 239.1 mm to (-94.7, 202.2)
- moved R12 238.8 mm to (-94.7, 204.2)
- moved D2 230.1 mm to (-98.7, 202.7)
- moved U4 230.1 mm to (-110.3, 203.3)
- moved C1 211.5 mm to (-101.4, 146.3)
- moved C2 211.5 mm to (-101.4, 149.0)
- moved R3 208.0 mm to (-52.0, 205.8)
- moved R4 208.0 mm to (-52.0, 207.8)
- moved C3 208.0 mm to (-48.6, 206.1)
- moved C4 208.0 mm to (-48.6, 208.7)
- moved R5 208.0 mm to (-52.0, 209.8)
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Connections:
- C1 pad 1: Net-(U1-VDD) -> +3.3V
- C1 pad 2: unconnected-(C1-Pad2) -> GND
- C2 pad 1: Net-(U1-VDD) -> +3.3V
- C2 pad 2: unconnected-(C2-Pad2) -> GND
- C5 pad 1: /Regulator DC/12V -> +12V
- C6 pad 1: /Regulator DC/3.3V -> +3.3V
- C7 pad 1: /Regulator DC/12V -> +12V
- C8 pad 1: /Regulator DC/5V -> +5V
- D1 pad 1: /Relay Motor/GND -> GND
- D2 pad 1: /RELAY/GND -> GND
- J1 pad 1: unconnected-(J1-Pin_1-Pad1) -> +3.3V
- J1 pad 4: unconnected-(J1-Pin_4-Pad4) -> GND
- J2 pad 1: /Relay Motor/5V -> /AC Trip/T1
- J2 pad 2: /Relay Motor/VDD -> /AC Trip/N
- J2 pad 3: /Relay Motor/12V -> /AC Trip/T2
- J6 pad 1: /HUMADITY/VCC -> +3.3V
- J6 pad 2: /HUMADITY/GND -> GND
- J6 pad 3: /HUMADITY/SCL -> /SCL
- J6 pad 4: /HUMADITY/SDA -> /SDA
- J6 pad 5: /HUMADITY/INT -> unconnected-(J6-Pin_5-Pad5)
- J7 pad 1: /Preasure & CO/V -> +3.3V
- J7 pad 2: /Preasure & CO/G -> GND
- J7 pad 3: /Preasure & CO/SCL -> /SCL
- J7 pad 4: /Preasure & CO/SDA -> /SDA
- J7 pad 5: unconnected-(J7-Pin_5-Pad5) -> +3.3V
- J7 pad 7: /Preasure & CO/A0 -> /D34
- J7 pad 8: /Preasure & CO/A1 -> /D35
- J8 pad 1: /Preasure & CO/GND -> GND
- J8 pad 2: /Preasure & CO/A1 -> /D35
- J8 pad 3: /Preasure & CO/5V -> +12V
- J9 pad 1: /Preasure & CO/5V -> +5V
- J9 pad 2: /Preasure & CO/A0 -> /D34
- J9 pad 3: /Preasure & CO/GND -> GND
- K1 pad 1: /Relay Motor/220V -> /Relay Motor1/220V
- K1 pad 3: /Relay Motor/MOTOR1 -> /Relay Motor1/MOTOR1
- K1 pad 5: /Relay Motor/VDD -> /VDD
- K2 pad 5: /RELAY/VOLT -> /VDD
- L1 pad 2: /Regulator DC/5V -> +5V
- R1 pad 1: /Relay Motor/PIN D -> /D27
- R11 pad 1: /RELAY/PIN D -> /D25
- R13 pad 1: /HUMADITY/3.3V -> +3.3V
- R13 pad 2: /HUMADITY/SCL -> /SCL
- R14 pad 1: /HUMADITY/3.3V -> +3.3V
- R14 pad 2: /HUMADITY/SDA -> /SDA
- R2 pad 1: Net-(R2-Pad1) -> /D28
- R3 pad 2: /SDcard/CS -> /CS
- R4 pad 1: +3.3V -> /MISO
- R4 pad 2: /SDcard/MOSI -> +3.3V
- R5 pad 1: +3.3V -> /CLK
- R5 pad 2: /SDcard/CLK -> +3.3V
- R6 pad 1: +3.3V -> /MOSI
- R6 pad 2: /SDcard/MISO -> +3.3V
- R7 pad 1: /rtc/3.3V -> +3.3V
- R7 pad 2: /rtc/SDA -> /SDA
- R8 pad 1: /rtc/3.3V -> +3.3V
- R8 pad 2: /rtc/SCL -> /SCL
- U1 pad 10: unconnected-(U1-IO25-Pad10) -> /D25
- U1 pad 11: unconnected-(U1-IO26-Pad11) -> /D26
- U1 pad 12: unconnected-(U1-IO27-Pad12) -> /D27
- U1 pad 14: unconnected-(U1-IO12-Pad14) -> /D12
- U1 pad 16: unconnected-(U1-IO13-Pad16) -> /D13
- U1 pad 2: Net-(U1-VDD) -> +3.3V
- U1 pad 23: unconnected-(U1-IO15-Pad23) -> /D15
- U1 pad 24: unconnected-(U1-IO2-Pad24) -> /D2
- U1 pad 25: unconnected-(U1-IO0-Pad25) -> Net-(J12-Pin_1)
- U1 pad 26: unconnected-(U1-IO4-Pad26) -> /D4
- U1 pad 27: unconnected-(U1-IO16-Pad27) -> /Tx
- U1 pad 28: unconnected-(U1-IO17-Pad28) -> /Rx
- U1 pad 29: unconnected-(U1-IO5-Pad29) -> /CS
- U1 pad 30: unconnected-(U1-IO18-Pad30) -> /SCK
- U1 pad 31: unconnected-(U1-IO19-Pad31) -> /MISO
- U1 pad 33: unconnected-(U1-IO21-Pad33) -> /SDA
- U1 pad 36: unconnected-(U1-IO22-Pad36) -> /SCL
- U1 pad 37: unconnected-(U1-IO23-Pad37) -> /MOSI
- U1 pad 6: unconnected-(U1-IO34-Pad6) -> /D34
- U1 pad 7: unconnected-(U1-IO35-Pad7) -> /D35
- U1 pad 8: unconnected-(U1-IO32-Pad8) -> /D28
- U1 pad 9: unconnected-(U1-IO33-Pad9) -> /D33
- U2 pad 3: Net-(R2-Pad1) -> Net-(R15-Pad1)
- U2 pad 4: /Relay Motor/VDD -> /VDD
- U3 pad 1: /LORA/GND -> GND
- U3 pad 12: /LORA/SCK -> /SCK
- U3 pad 13: /LORA/MISO -> /MISO
- U3 pad 14: /LORA/MOSI -> /MOSI
- U3 pad 15: /LORA/NSS -> /CS
- U3 pad 16: /LORA/GND -> GND
- U3 pad 2: /LORA/GND -> GND
- U3 pad 3: /LORA/3V3 -> +3.3V
- U3 pad 4: /LORA/RST -> /D15
- U3 pad 5: /LORA/PIN D -> /D33
- U3 pad 9: /LORA/GND -> GND
- U4 pad 4: /RELAY/VOLT -> /VDD
- U5 pad 2: /Regulator DC/3.3V -> +3.3V
- U5 pad 3: /Regulator DC/12V -> +12V
- U6 pad 1: /Regulator DC/12V -> +12V
- U6 pad 4: /Regulator DC/5V -> +5V
- U7 pad 10: /rtc/GND -> GND
- U7 pad 11: /rtc/GND -> GND
- U7 pad 12: /rtc/GND -> GND
- U7 pad 13: /rtc/GND -> GND
- U7 pad 14: unconnected-(U7-VBAT-Pad14) -> Net-(BAT1-+)
- U7 pad 15: /rtc/SDA -> /SDA
- U7 pad 16: /rtc/SCL -> /SCL
- U7 pad 2: /rtc/3.3V -> +3.3V
- U7 pad 5: /rtc/GND -> GND
- U7 pad 6: /rtc/GND -> GND
- U7 pad 7: /rtc/GND -> GND
- U7 pad 8: /rtc/GND -> GND
- U7 pad 9: /rtc/GND -> GND

Commit message: menghapus file tidak perlu
Parts:
- added BT1: CR1220MFR_FH, CR1220:CR1220-SMD, F.Cu at (-117.2, 92.5)
- added J3: MSD-4-A, MSD-4-A:CUI_MSD-4-A, F.Cu at (-126.0, 121.5)
- added Q1: 2N5551-TA, Package_TO_SOT_THT:TO-92_Inline_Wide, F.Cu at (-44.5, 108.8)
- added Q2: 2N5551-TA, Package_TO_SOT_THT:TO-92_Inline_Wide, F.Cu at (-18.7, 134.7)
- added Q3: 2N5551-TA, Package_TO_SOT_THT:TO-92_Inline_Wide, F.Cu at (-44.5, 134.7)
- added Q4: 2N5551-TA, Package_TO_SOT_THT:TO-92_Inline_Wide, F.Cu at (-18.7, 108.8)
- U3: footprint RA-02_LORA:MODULE_RA-02_LORA -> RF_Module:Ai-Thinker-Ra-01-LoRa
- moved U7 241.1 mm to (-98.7, 109.0)
- moved U3 233.1 mm to (-95.4, 126.5), turned to 0 degrees
- moved U1 219.2 mm to (-94.9, 75.7)
- moved U6 200.0 mm to (-24.6, 59.4)
- moved J17 197.2 mm to (213.9, 74.5), turned to -90 degrees
- moved J15 195.2 mm to (214.0, 134.0), turned to -90 degrees
- moved J16 195.0 mm to (213.9, 94.0), turned to -90 degrees
- moved J18 195.0 mm to (213.9, 115.0)
- moved J8 166.1 mm to (-46.0, 65.1)
- moved J7 164.2 mm to (-51.7, 55.6), turned to 0 degrees
- moved K4 162.7 mm to (188.5, 76.0)
- moved K2 160.7 mm to (188.6, 116.0)
- moved K3 160.7 mm to (188.5, 96.0)
- moved K1 160.1 mm to (188.5, 136.5)
- moved J9 154.8 mm to (-45.9, 57.5)
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